File: Eagle/Cerradura electronica/Cerradura electronica.sch (EAGLE design)
At the start: 38 parts, among them IC1 LD117AS50TR, Q1 2N3904, Q2 IRF540NS, U1 ATMEGA328P_TQFP

Commit message: Etapa de potencia con activacion GPS y teclado simultanea
Parts:
- R7: value 1k -> 150R
Changed lines of the file:
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@@
 <grid distance="0.1" unitdist="inch" unit="inch" style="lines" multiple="1" display="no" altdistance="0.01" altunitdist="inch" altunit="inch"/>
 <layers>
-<layer number="1" name="Top" color="4" fill="1" visible="yes" active="no"/>
-<layer number="2" name="Route2" color="1" fill="3" visible="yes" active="no"/>
-<layer number="3" name="Route3" color="4" fill="3" visible="yes" active="no"/>
-<layer number="4" name="Route4" color="1" fill="4" visible="yes" active="no"/>
-<layer number="5" name="Route5" color="4" fill="4" visible="yes" active="no"/>
-<layer number="6" name="Route6" color="1" fill="8" visible="yes" active="no"/>
-<layer number="7" name="Route7" color="4" fill="8" visible="yes" active="no"/>
-<layer number="8" name="Route8" color="1" fill="2" visible="yes" active="no"/>
-<layer number="9" name="Route9" color="4" fill="2" visible="yes" active="no"/>
-<layer number="10" name="Route10" color="1" fill="7" visible="yes" active="no"/>
-<layer number="11" name="Route11" color="4" fill="7" visible="yes" active="no"/>
-<layer number="12" name="Route12" color="1" fill="5" visible="yes" active="no"/>
-<layer number="13" name="Route13" color="4" fill="5" visible="yes" active="no"/>
-<layer number="14" name="Route14" color="1" fill="6" visible="yes" active="no"/>
-<layer number="15" name="Route15" color="4" fill="6" visible="yes" active="no"/>
-<layer number="16" name="Bottom" color="1" fill="1" visible="yes" active="no"/>
-<layer number="17" name="Pads" color="2" fill="1" visible="yes" active="no"/>
-<layer number="18" name="Vias" color="2" fill="1" visible="yes" active="no"/>
-<layer number="19" name="Unrouted" color="6" fill="1" visible="yes" active="no"/>
-<layer number="20" name="Dimension" color="15" fill="1" visible="yes" active="no"/>
-<layer number="21" name="tPlace" color="61" fill="1" visible="yes" active="no"/>
-<layer number="22" name="bPlace" color="63" fill="1" visible="yes" active="no"/>
-<layer number="23" name="tOrigins" color="15" fill="1" visible="yes" active="no"/>
-<layer number="24" name="bOrigins" color="15" fill="1" visible="yes" active="no"/>
-<layer number="25" name="tNames" color="11" fill="1" visible="yes" active="no"/>
-<layer number="26" name="bNames" color="7" fill="1" visible="yes" active="no"/>
-<layer number="27" name="tValues" color="7" fill="1" visible="yes" active="no"/>
-<layer number="28" name="bValues" color="7" fill="1" visible="yes" active="no"/>
+<layer number="1" name="Top" color="4" fill="1" visible="no" active="no"/>
+<layer number="2" name="Route2" color="1" fill="3" visible="no" active="no"/>
+<layer number="3" name="Route3" color="4" fill="3" visible="no" active="no"/>
+<layer number="4" name="Route4" color="1" fill="4" visible="no" active="no"/>
+<layer number="5" name="Route5" color="4" fill="4" visible="no" active="no"/>
+<layer number="6" name="Route6" color="1" fill="8" visible="no" active="no"/>
+<layer number="7" name="Route7" color="4" fill="8" visible="no" active="no"/>
+<layer number="8" name="Route8" color="1" fill="2" visible="no" active="no"/>
+<layer number="9" name="Route9" color="4" fill="2" visible="no" active="no"/>
+<layer number="10" name="Route10" color="1" fill="7" visible="no" active="no"/>
+<layer number="11" name="Route11" color="4" fill="7" visible="no" active="no"/>
+<layer number="12" name="Route12" color="1" fill="5" visible="no" active="no"/>
+<layer number="13" name="Route13" color="4" fill="5" visible="no" active="no"/>
+<layer number="14" name="Route14" color="1" fill="6" visible="no" active="no"/>
+<layer number="15" name="Route15" color="4" fill="6" visible="no" active="no"/>
+<layer number="16" name="Bottom" color="1" fill="1" visible="no" active="no"/>
+<layer number="17" name="Pads" color="2" fill="1" visible="no" active="no"/>
+<layer number="18" name="Vias" color="2" fill="1" visible="no" active="no"/>
+<layer number="19" name="Unrouted" color="6" fill="1" visible="no" active="no"/>
+<layer number="20" name="Dimension" color="15" fill="1" visible="no" active="no"/>
+<layer number="21" name="tPlace" color="61" fill="1" visible="no" active="no"/>
+<layer number="22" name="bPlace" color="63" fill="1" visible="no" active="no"/>
+<layer number="23" name="tOrigins" color="15" fill="1" visible="no" active="no"/>
+<layer number="24" name="bOrigins" color="15" fill="1" visible="no" active="no"/>
+<layer number="25" name="tNames" color="11" fill="1" visible="no" active="no"/>
+<layer number="26" name="bNames" color="7" fill="1" visible="no" active="no"/>
+<layer number="27" name="tValues" color="7" fill="1" visible="no" active="no"/>
+<layer number="28" name="bValues" color="7" fill="1" visible="no" active="no"/>
 <layer number="29" name="tStop" color="7" fill="3" visible="no" active="no"/>
 <layer number="30" name="bStop" color="7" fill="6" visible="no" active="no"/>
@@
 <layer number="35" name="tGlue" color="7" fill="4" visible="no" active="no"/>
 <layer number="36" name="bGlue" color="7" fill="5" visible="no" active="no"/>
-<layer number="37" name="tTest" color="7" fill="1" visible="yes" active="no"/>
-<layer number="38" name="bTest" color="7" fill="1" visible="yes" active="no"/>
+<layer number="37" name="tTest" color="7" fill="1" visible="no" active="no"/>
+<layer number="38" name="bTest" color="7" fill="1" visible="no" active="no"/>
 <layer number="39" name="tKeepout" color="4" fill="11" visible="no" active="no"/>
 <layer number="40" name="bKeepout" color="1" fill="11" visible="no" active="no"/>
@@
 <layer number="44" name="Drills" color="7" fill="1" visible="no" active="no"/>
 <layer number="45" name="Holes" color="7" fill="1" visible="no" active="no"/>
-<layer number="46" name="Milling" color="3" fill="1" visible="yes" active="no"/>
-<layer number="47" name="Measures" color="17" fill="1" visible="yes" active="no"/>
-<layer number="48" name="Document" color="7" fill="1" visible="yes" active="no"/>
-<layer number="49" name="Reference" color="7" fill="1" visible="yes" active="no"/>
-<layer number="50" name="dxf" color="7" fill="1" visible="yes" active="no"/>
-<layer number="51" name="tDocu" color="7" fill="1" visible="yes" active="no"/>
-<layer number="52" name="bDocu" color="7" fill="1" visible="yes" active="no"/>
-<layer number="53" name="tGND_GNDA" color="7" fill="9" visible="yes" active="no"/>
-<layer number="54" name="bGND_GNDA" color="1" fill="9" visible="yes" active="no"/>
-<layer number="56" name="wert" color="7" fill="1" visible="yes" active="no"/>
-<layer number="57" name="tCAD" color="7" fill="1" visible="yes" active="no"/>
-<layer number="59" name="tCarbon" color="7" fill="1" visible="yes" active="no"/>
-<layer number="60" name="bCarbon" color="7" fill="1" visible="yes" active="no"/>
+<layer number="46" name="Milling" color="3" fill="1" visible="no" active="no"/>
+<layer number="47" name="Measures" color="17" fill="1" visible="no" active="no"/>
+<layer number="48" name="Document" color="7" fill="1" visible="no" active="no"/>
+<layer number="49" name="Reference" color="7" fill="1" visible="no" active="no"/>
+<layer number="50" name="dxf" color="7" fill="1" visible="no" active="no"/>
+<layer number="51" name="tDocu" color="7" fill="1" visible="no" active="no"/>
+<layer number="52" name="bDocu" color="7" fill="1" visible="no" active="no"/>
+<layer number="53" name="tGND_GNDA" color="7" fill="9" visible="no" active="no"/>
+<layer number="54" name="bGND_GNDA" color="1" fill="9" visible="no" active="no"/>
+<layer number="56" name="wert" color="7" fill="1" visible="no" active="no"/>
+<layer number="57" name="tCAD" color="7" fill="1" visible="no" active="no"/>
+<layer number="59" name="tCarbon" color="7" fill="1" visible="no" active="no"/>
+<layer number="60" name="bCarbon" color="7" fill="1" visible="no" active="no"/>
 <layer number="90" name="Modules" color="5" fill="1" visible="yes" active="yes"/>
 <layer number="91" name="Nets" color="2" fill="1" visible="yes" active="yes"/>
@@
 <part name="R2" library="rcl" deviceset="R-US_" device="R1206" value="1k"/>
 <part name="PWR" library="con-ptr500" deviceset="AK500/2" device=""/>
-<part name="R7" library="rcl" deviceset="R-US_" device="R1206" value="1k"/>
+<part name="R7" library="rcl" deviceset="R-US_" device="R1206" value="150R"/>
 <part name="R8" library="rcl" deviceset="R-US_" device="R1206" value="10k"/>
 <part name="P+1" library="supply1" deviceset="VCC" device=""/>

Commit message: Inicio correciones en PCB
Parts:
- added D3: MBRA340T3, diode:MBRA340T3
- C1, C12, C2, C3, C4, C5, C6, C7, C8, C9: device rcl:C-USC0805 -> CaliBeta-RCL:CAPC0805
- C10, C11: device rcl:C-USC1206 -> CaliBeta-RCL:CAPC1206
- D1, D2: device diode:DIODE-DO214AC -> CaliBeta-Diodos:DIODO-DO-214AC
- ISP: value (none) -> CON-ISP; device con-lstb:MA03-2 -> CaliBeta-Conectores:CON-ISP
- L1: device Circuitos-Creativos-RCL:FERRITA-CHOKE -> CaliBeta-RCL:IND-FER-L0805
- LED1: value Green -> Rojo; device led:LEDCHIPLED_0805 -> CaliBeta-Diodos:LED-ROJO0805
- MOT, PWR: device con-ptr500:AK500/2 -> CaliBeta-Conectores:AK500-2
- Q1: device transistor:MMBT3904LT1-NPN-SOT23-BEC -> CaliBeta-Transistores:SS8050
- Q2: value IRF540NS -> IRF540N; device Circuitos-Creativos-Transistores:IRF540NS -> CaliBeta-Transistores:IRF540N
- R1, R2, R3, R4, R5, R6, R7, R8: device rcl:R-US_R1206 -> CaliBeta-RCL:RESISTOR_R0805
- R10, R9: device rcl:R-US_R1206 -> CaliBeta-RCL:RESISTOR_R1206
- U1: value ATMEGA328P_TQFP -> (none); device SparkFun-DigitalIC:ATMEGA328P_TQFP -> CaliBeta-Microcontroladores:ATMEGA328P-AU
Connections:
- removed net MOT_ON: C12.2, D2.A, MOT-2.KL, Q2.D
- new net MOT: D3.A, MOT-1.KL1
- new net ON: C12.2, D2.A, D3.C, Q2.D
- net +12V: now also MOT-2.KL1, PWR-1.KL1; no longer MOT-1.KL, PWR-2.KL
- net GND: now also PWR-2.KL1, U1.GND; no longer PWR-1.KL, U1.GND@3, U1.GND@5
- net OS1: now also U1.PB6(XTAL1/TOSC1); no longer U1.PB6(XTAL1)
- net OS2: now also U1.PB7(XTAL2/TOSC2); no longer U1.PB7(XTAL2)
- net VCC: now also U1.VCC; no longer U1.VCC@4, U1.VCC@6
Other:
- note added: "1.5"
- note removed: "1.1"
- moved on the sheet: C1, C10, C11, C2, C5, IC1, L1, LED1, MOT-1, MOT-2, PWR-1, PWR-2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
