File: Eagle/Cerradura electronica/Cerradura electronica.sch (EAGLE design)
At the start: 39 parts, among them IC1 LD117AS50TR, Q1 2N3904, Q2 IRF540N

Commit message: correciones en PCB al 75%
Parts:
- removed C1, C2: 22pF, CaliBeta-RCL:CAPC0805
- removed XT2: 8MHz, crystal:CRYSTALSM49
- added XT1: 8MHz, CaliBeta-Miselaneos:CRISTAL-3215
- R10, R9: device CaliBeta-RCL:RESISTOR_R1206 -> CaliBeta-RCL:RESISTOR_R0805
Connections:
- removed net OS1: C1.1, U1.PB6(XTAL1/TOSC1), XT2.2
- removed net OS2: C2.1, U1.PB7(XTAL2/TOSC2), XT2.1
- new net N$5: U1.PB6(XTAL1/TOSC1), XT1.X1
- new net N$6: U1.PB7(XTAL2/TOSC2), XT1.X2
- net GND: now also XT1.GND; no longer C1.2, C2.2
Changed lines of the file:
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@@
 <part name="GND9" library="SparkFun" deviceset="GND" device=""/>
 <part name="GND10" library="SparkFun" deviceset="GND" device=""/>
-<part name="GND11" library="SparkFun" deviceset="GND" device=""/>
 <part name="P+15" library="supply1" library_urn="urn:adsk.eagle:library:371" deviceset="VCC" device=""/>
 <part name="P+4" library="supply1" library_urn="urn:adsk.eagle:library:371" deviceset="VCC" device=""/>
@@
 <part name="C3" library="CaliBeta-RCL" library_urn="urn:adsk.eagle:library:14345719" deviceset="CAP" device="C0805" package3d_urn="urn:adsk.eagle:package:14345754/1" value="0.1uF"/>
 <part name="C4" library="CaliBeta-RCL" library_urn="urn:adsk.eagle:library:14345719" deviceset="CAP" device="C0805" package3d_urn="urn:adsk.eagle:package:14345754/1" value="0.1uF"/>
-<part name="XT2" library="crystal" library_urn="urn:adsk.eagle:library:204" deviceset="CRYSTAL" device="SM49" package3d_urn="urn:adsk.eagle:package:12085/1" value="8MHz"/>
-<part name="C1" library="CaliBeta-RCL" library_urn="urn:adsk.eagle:library:14345719" deviceset="CAP" device="C0805" package3d_urn="urn:adsk.eagle:package:14345754/1" value="22pF"/>
-<part name="C2" library="CaliBeta-RCL" library_urn="urn:adsk.eagle:library:14345719" deviceset="CAP" device="C0805" package3d_urn="urn:adsk.eagle:package:14345754/1" value="22pF"/>
-<part name="GND24" library="SparkFun" deviceset="GND" device=""/>
 <part name="ISP" library="CaliBeta-Conectores" library_urn="urn:adsk.eagle:library:14344905" deviceset="CON-ISP" device="" package3d_urn="urn:adsk.eagle:package:14344941/1"/>
 <part name="L1" library="CaliBeta-RCL" library_urn="urn:adsk.eagle:library:14345719" deviceset="IND-FER-" device="L0805" package3d_urn="urn:adsk.eagle:package:14345752/2" value="10u"/>
@@
 <part name="P+1" library="supply1" library_urn="urn:adsk.eagle:library:371" deviceset="VCC" device=""/>
 <part name="D1" library="CaliBeta-Diodos" library_urn="urn:adsk.eagle:library:14345451" deviceset="DIODO" device="-DO-214AC" package3d_urn="urn:adsk.eagle:package:14345492/2" value="4004"/>
-<part name="R9" library="CaliBeta-RCL" library_urn="urn:adsk.eagle:library:14345719" deviceset="RESISTOR_" device="R1206" package3d_urn="urn:adsk.eagle:package:14345748/2" value="10k"/>
+<part name="R9" library="CaliBeta-RCL" library_urn="urn:adsk.eagle:library:14345719" deviceset="RESISTOR_" device="R0805" package3d_urn="urn:adsk.eagle:package:14345749/1" value="10k"/>
 <part name="P+2" library="supply1" library_urn="urn:adsk.eagle:library:371" deviceset="+12V" device=""/>
 <part name="GND15" library="supply1" library_urn="urn:adsk.eagle:library:371" deviceset="GND" device=""/>
@@
 <part name="P+3" library="supply1" library_urn="urn:adsk.eagle:library:371" deviceset="+12V" device=""/>
 <part name="TECLADO" library="con-lstb" library_urn="urn:adsk.eagle:library:162" deviceset="MA07-1" device="" package3d_urn="urn:adsk.eagle:package:8341/1"/>
-<part name="R10" library="CaliBeta-RCL" library_urn="urn:adsk.eagle:library:14345719" deviceset="RESISTOR_" device="R1206" package3d_urn="urn:adsk.eagle:package:14345748/2" value="1k"/>
+<part name="R10" library="CaliBeta-RCL" library_urn="urn:adsk.eagle:library:14345719" deviceset="RESISTOR_" device="R0805" package3d_urn="urn:adsk.eagle:package:14345749/1" value="1k"/>
 <part name="P+6" library="supply1" library_urn="urn:adsk.eagle:library:371" deviceset="VCC" device=""/>
 <part name="GND17" library="SparkFun" deviceset="GND" device=""/>
@@
 <part name="P+7" library="supply1" library_urn="urn:adsk.eagle:library:371" deviceset="VCC" device=""/>
 <part name="GND12" library="SparkFun" deviceset="GND" device=""/>
+<part name="XT1" library="CaliBeta-Miselaneos" library_urn="urn:adsk.eagle:library:14357685" deviceset="CRISTAL-3215" device="" package3d_urn="urn:adsk.eagle:package:14357744/1" value="8MHz"/>
+<part name="GND11" library="SparkFun" deviceset="GND" device=""/>
 </parts>
 <sheets>
@@
 <attribute name="VALUE" x="50.8" y="55.88" size="1.778" layer="96" ratio="10"/>
 </instance>
-<instance part="GND11" gate="1" x="5.08" y="127" smashed="yes" rot="R270">
-<attribute name="VALUE" x="2.54" y="129.54" size="1.778" layer="96" ratio="10" rot="R270"/>
-</instance>
 <instance part="P+15" gate="VCC" x="7.62" y="96.52" smashed="yes">
 <attribute name="VALUE" x="10.16" y="99.06" size="1.778" layer="96" ratio="10" rot="R180"/>
@@
 <attribute name="NAME" x="57.404" y="70.993" size="1.778" layer="95" ratio="10" rot="R180"/>
 <attribute name="VALUE" x="54.356" y="63.881" size="1.778" layer="96" ratio="10"/>
-</instance>
-<instance part="XT2" gate="G$1" x="22.86" y="132.08" smashed="yes" rot="R90">
-<attribute name="NAME" x="23.368" y="134.366" size="1.778" layer="95" ratio="10"/>
-<attribute name="VALUE" x="20.32" y="128.524" size="1.778" layer="96" ratio="10" rot="R90"/>
-</instance>
-<instance part="C1" gate="G$1" x="15.24" y="137.16" smashed="yes" rot="R270">
-<attribute name="NAME" x="16.764" y="142.113" size="1.778" layer="95" ratio="10" rot="R180"/>
-<attribute name="VALUE" x="11.176" y="132.461" size="1.778" layer="96" ratio="10"/>
-</instance>
-<instance part="C2" gate="G$1" x="15.24" y="127" smashed="yes" rot="R270">
-<attribute name="NAME" x="16.764" y="131.953" size="1.778" layer="95" ratio="10" rot="R180"/>
-<attribute name="VALUE" x="11.176" y="122.301" size="1.778" layer="96" ratio="10"/>
-</instance>
-<instance part="GND24" gate="1" x="5.08" y="137.16" smashed="yes" rot="R270">
-<attribute name="VALUE" x="2.54" y="139.7" size="1.778" layer="96" ratio="10" rot="R270"/>
 </instance>
 <instance part="ISP" gate="G$1" x="25.4" y="66.04" smashed="yes">
@@
 <instance part="GND12" gate="1" x="50.8" y="81.28" smashed="yes">
 <attribute name="VALUE" x="48.26" y="78.74" size="1.778" layer="96" ratio="10"/>
+</instance>
+<instance part="XT1" gate="G$1" x="17.78" y="132.08" smashed="yes">
+<attribute name="NAME" x="15.24" y="138.684" size="1.778" layer="95"/>
+<attribute name="VALUE" x="15.24" y="123.698" size="1.778" layer="96"/>
+</instance>
+<instance part="GND11" gate="1" x="7.62" y="132.08" smashed="yes" rot="R270">
+<attribute name="VALUE" x="5.08" y="134.62" size="1.778" layer="96" ratio="10" rot="R270"/>
 </instance>
 </instances>
@@
 <pinref part="SV1" gate="1" pin="4"/>
 <wire x1="78.74" y1="63.5" x2="81.28" y2="63.5" width="0.1524" layer="91"/>
-</segment>
-<segment>
-<pinref part="C2" gate="G$1" pin="2"/>
-<pinref part="GND11" gate="1" pin="GND"/>
-<wire x1="7.62" y1="127" x2="10.16" y2="127" width="0.1524" layer="91"/>
-</segment>
-<segment>
-<pinref part="GND24" gate="1" pin="GND"/>
-<pinref part="C1" gate="G$1" pin="2"/>
-<wire x1="7.62" y1="137.16" x2="10.16" y2="137.16" width="0.1524" layer="91"/>
 </segment>
 <segment>
@@
 <pinref part="GND12" gate="1" pin="GND"/>
 <wire x1="50.8" y1="83.82" x2="50.8" y2="86.36" width="0.1524" layer="91"/>
+</segment>
+<segment>
+<pinref part="XT1" gate="G$1" pin="GND"/>
+<pinref part="GND11" gate="1" pin="GND"/>
+<wire x1="10.16" y1="132.08" x2="12.7" y2="132.08" width="0.1524" layer="91"/>
 </segment>
 </net>
@@
 <label x="81.28" y="99.06" size="1.27" layer="95" ratio="10" xref="yes"/>
 <pinref part="U1" gate="G$1" pin="PB2(SS/OC1B)"/>
-</segment>
-</net>
-<net name="OS2" class="0">
-<segment>
-<pinref part="C2" gate="G$1" pin="1"/>
-<wire x1="25.4" y1="127" x2="22.86" y2="127" width="0.1524" layer="91"/>
-<pinref part="XT2" gate="G$1" pin="1"/>
-<wire x1="22.86" y1="127" x2="17.78" y2="127" width="0.1524" layer="91"/>
-<wire x1="22.86" y1="129.54" x2="22.86" y2="127" width="0.1524" layer="91"/>
-<junction x="22.86" y="127"/>
-<pinref part="U1" gate="G$1" pin="PB7(XTAL2/TOSC2)"/>
-</segment>
-</net>
-<net name="OS1" class="0">
-<segment>
-<pinref part="C1" gate="G$1" pin="1"/>
-<pinref part="XT2" gate="G$1" pin="2"/>
-<wire x1="22.86" y1="137.16" x2="17.78" y2="137.16" width="0.1524" layer="91"/>
-<wire x1="22.86" y1="134.62" x2="22.86" y2="137.16" width="0.1524" layer="91"/>
-<wire x1="25.4" y1="137.16" x2="22.86" y2="137.16" width="0.1524" layer="91"/>
-<junction x="22.86" y="137.16"/>
-<pinref part="U1" gate="G$1" pin="PB6(XTAL1/TOSC1)"/>
 </segment>
 </net>
@@
 </segment>
 </net>
+<net name="N$5" class="0">
+<segment>
+<pinref part="U1" gate="G$1" pin="PB6(XTAL1/TOSC1)"/>
+<pinref part="XT1" gate="G$1" pin="X1"/>
+<wire x1="22.86" y1="137.16" x2="25.4" y2="137.16" width="0.1524" layer="91"/>
+</segment>
+</net>
+<net name="N$6" class="0">
+<segment>
+<pinref part="U1" gate="G$1" pin="PB7(XTAL2/TOSC2)"/>
+<pinref part="XT1" gate="G$1" pin="X2"/>
+<wire x1="22.86" y1="127" x2="25.4" y2="127" width="0.1524" layer="91"/>
+</segment>
+</net>

Commit message: Terminado correciones
Parts:
- S1: device Testing:SWITCH-MOMENTARY-2-SMD-1101NE -> CaliBeta-Miselaneos:PULSADOR-SMD-6035
- XT1: device CaliBeta-Miselaneos:CRISTAL-3215 -> CaliBeta-Miselaneos:XTAL-CSTCE
Connections:
- net GND: now also S1.P$1; no longer S1.1
- net RST: now also S1.P$2; no longer S1.2
Changed lines of the file:
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@@
 <part name="P+6" library="supply1" library_urn="urn:adsk.eagle:library:371" deviceset="VCC" device=""/>
 <part name="GND17" library="SparkFun" deviceset="GND" device=""/>
-<part name="S1" library="Testing" deviceset="SWITCH-MOMENTARY-2" device="-SMD-1101NE" value="Reset"/>
+<part name="S1" library="CaliBeta-Miselaneos" library_urn="urn:adsk.eagle:library:14357685" deviceset="PULSADOR-" device="SMD-6035" package3d_urn="urn:adsk.eagle:package:14566828/2" value="Reset"/>
 <part name="P+5" library="supply1" library_urn="urn:adsk.eagle:library:371" deviceset="VCC" device=""/>
 <part name="GND18" library="supply1" library_urn="urn:adsk.eagle:library:371" deviceset="GND" device=""/>
@@
 <part name="P+7" library="supply1" library_urn="urn:adsk.eagle:library:371" deviceset="VCC" device=""/>
 <part name="GND12" library="SparkFun" deviceset="GND" device=""/>
-<part name="XT1" library="CaliBeta-Miselaneos" library_urn="urn:adsk.eagle:library:14357685" deviceset="CRISTAL-3215" device="" package3d_urn="urn:adsk.eagle:package:14357744/1" value="8MHz"/>
+<part name="XT1" library="CaliBeta-Miselaneos" library_urn="urn:adsk.eagle:library:14357685" deviceset="XTAL-" device="CSTCE" package3d_urn="urn:adsk.eagle:package:14357744/2" value="8MHz"/>
 <part name="GND11" library="SparkFun" deviceset="GND" device=""/>
 </parts>
@@
 <attribute name="VALUE" x="40.64" y="157.48" size="1.778" layer="96" rot="R90"/>
 </instance>
-<instance part="S1" gate="G$1" x="25.4" y="160.02" smashed="yes" rot="R180">
+<instance part="S1" gate="P1" x="25.4" y="160.02" smashed="yes" rot="R180">
 <attribute name="NAME" x="25.4" y="157.48" size="1.778" layer="95" rot="R180"/>
 <attribute name="VALUE" x="27.94" y="162.56" size="1.778" layer="96" rot="R180"/>
@@
 <wire x1="30.48" y1="160.02" x2="35.56" y2="160.02" width="0.1524" layer="91"/>
 <pinref part="GND17" gate="1" pin="GND"/>
-<pinref part="S1" gate="G$1" pin="1"/>
+<pinref part="S1" gate="P1" pin="P$1"/>
 </segment>
 <segment>
@@
 <segment>
 <wire x1="20.32" y1="160.02" x2="10.16" y2="149.86" width="0.1524" layer="91"/>
-<pinref part="S1" gate="G$1" pin="2"/>
+<pinref part="S1" gate="P1" pin="P$2"/>
 <wire x1="25.4" y1="149.86" x2="10.16" y2="149.86" width="0.1524" layer="91"/>
 <pinref part="R1" gate="G$1" pin="2"/>
