File: Eagle/Cerradura electronica/Cerradura electronica.brd (EAGLE design)
At the start: 48.5 x 50 mm, 38 parts, among them IC1 LD117AS50TR, Q1 2N3904, Q2 IRF540NS, U1 ATMEGA328P_TQFP

Commit message: Inicio correciones en PCB
Parts:
- added D3: MBRA340T3, diode:SMA
- C1, C12, C2, C3, C4, C5, C6, C7, C8, C9: device rcl:C0805 -> CaliBeta-RCL:C0805
- C10, C11: device rcl:C1206 -> CaliBeta-RCL:C1206
- D1, D2: device diode:DO214AC -> CaliBeta-Diodos:DO-214AC
- ISP: value (none) -> CON-ISP; device con-lstb:MA03-2 -> CaliBeta-Conectores:HEADER-M2X3
- L1: device Circuitos-Creativos-RCL:L0805 -> CaliBeta-RCL:L0805
- LED1: value Green -> Rojo; device led:CHIPLED_0805 -> CaliBeta-Diodos:LED0805-ROJO
- MOT, PWR: device con-ptr500:AK500/2 -> CaliBeta-Conectores:AK500-2
- Q1: device transistor:SOT23-BEC -> CaliBeta-Transistores:SOT-23_BEC
- Q2: value IRF540NS -> IRF540N; device Circuitos-Creativos-Transistores:TO-252 -> CaliBeta-Transistores:TO-263
- R1, R2, R3, R4, R5, R6, R7, R8: device rcl:R1206 -> CaliBeta-RCL:R0805
- R10, R9: device rcl:R1206 -> CaliBeta-RCL:R1206
- U1: value ATMEGA328P_TQFP -> (none); device SparkFun-DigitalIC:TQFP32-08 -> CaliBeta-Microcontroladores:TQFP32
- moved C7 37.7 mm to (42.5, 44.0), turned to 90 degrees
- moved D2 36.7 mm to (3.00, 39.0), turned to 270 degrees
- moved C2 35.6 mm to (47.5, 36.0), turned to 0 degrees
- moved R4 35.4 mm to (39.8, 44.0), turned to 90 degrees
- moved MOT 34.2 mm to (11.5, 45.0), turned to 180 degrees
- moved D1 34.0 mm to (3.00, 14.5), turned to 270 degrees
- moved C6 33.5 mm to (37.0, 44.0), turned to 90 degrees
- moved U$1 33.3 mm to (44.0, 11.2), turned to 270 degrees
- moved PWR 33.2 mm to (11.5, 4.50), turned to 0 degrees
- moved C1 32.9 mm to (47.5, 31.0), turned to 0 degrees
- moved R3 32.0 mm to (34.2, 44.0), turned to 90 degrees
- moved SV1 31.6 mm to (47.0, 22.5), turned to 270 degrees
- moved C9 31.0 mm to (31.5, 44.0), turned to 90 degrees
- moved R5 31.0 mm to (23.2, 44.0), turned to 90 degrees
- moved R6 30.4 mm to (28.8, 44.0), turned to 90 degrees
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Connections:
- removed net MOT_ON: C12.2, D2.A, MOT.2, Q2.3
- new net MOT: D3.A, MOT.1
- new net ON: C12.2, D2.A, D3.C, Q2.2
- net +12V: now also D2.K, MOT.2, PWR.1; no longer D2.C, MOT.1, PWR.2
- net GND: now also PWR.2, Q2.3; no longer PWR.1, Q2.2
- net N$3: now also D1.K; no longer D1.C
Routing:
- net GND: track 249.1 -> 138.2 mm, vias 3 -> 1
- net D3: track 34.2 -> 0.00 mm, vias 2 -> 0
- net RST: track 70.4 -> 36.5 mm
- net +12V: track 111.3 -> 81.7 mm, vias 5 -> 4
- net VCC: track 125.3 -> 96.0 mm, vias 5 -> 4
- net ON: track 0.00 -> 29.3 mm
- net MOT_ON: track 25.9 -> 0.00 mm, vias 1 -> 0
- net D8/3: track 23.0 -> 9.64 mm
- net D5/2: track 17.8 -> 5.49 mm
- net N$2: track 12.1 -> 0.00 mm
- net MOSI: track 14.8 -> 3.78 mm, vias 1 -> 0
- net D7/4: track 19.4 -> 8.81 mm
- net D6/1: track 16.3 -> 6.21 mm
- net MOT: track 0.00 -> 5.90 mm
- net N$4: track 9.09 -> 13.5 mm
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Other:
- board size 48.5 x 50 mm -> 50 x 48.5 mm

Commit message: correciones en PCB al 75%
Parts:
- removed C1, C2: 22pF, CaliBeta-RCL:C0805
- removed XT2: 8MHz, crystal:SM49
- added XT1: 8MHz, CaliBeta-Miselaneos:CSTCE8M00G55-R0
- R10, R9: device CaliBeta-RCL:R1206 -> CaliBeta-RCL:R0805
- moved C3 9.01 mm to (42.5, 27.5), turned to 90 degrees
- moved TECLADO 4.03 mm to (33.0, 38.0)
- moved C10 1.12 mm to (32.5, 13.5)
- moved R1 1.12 mm to (37.0, 13.5)
- moved LED1 1.00 mm to (26.5, 13.5)
- moved R2 1.00 mm to (23.0, 13.5)
- moved R7 1.00 mm to (19.0, 13.5), turned to 90 degrees
- moved S1 0.71 mm to (34.5, 20.0)
- moved C11 0.50 mm to (23.0, 20.0)
- moved C4 0.50 mm to (26.5, 20.0)
- moved C5 0.50 mm to (26.5, 27.0)
- moved L1 0.50 mm to (26.5, 32.0)
- moved R10 0.50 mm to (14.5, 37.0)
- moved R8 0.50 mm to (19.0, 20.0)
- moved SV1 0.38 mm to (46.6, 22.5)
Connections:
- removed net OS1: C1.1, U1.7, XT2.2
- removed net OS2: C2.1, U1.8, XT2.1
- new net N$5: U1.7, XT1.1
- new net N$6: U1.8, XT1.3
- net GND: now also XT1.2; no longer C1.2, C2.2
Routing:
- net VCC: track 96.0 -> 34.8 mm, vias 4 -> 1
- net +12V: track 81.7 -> 105.5 mm
- net OS2: track 14.3 -> 0.00 mm
- net GND: track 138.2 -> 151.8 mm, vias 1 -> 0
- net N$2: track 0.00 -> 13.1 mm
- net D5/2: track 5.49 -> 18.3 mm
- net D8/3: track 9.64 -> 22.1 mm
- net OS1: track 11.0 -> 0.00 mm
- net MOSI: track 3.78 -> 13.1 mm, vias 0 -> 1
- net D7/4: track 8.81 -> 17.4 mm
- net RST: track 36.5 -> 28.6 mm
- net D6/1: track 6.21 -> 13.6 mm
- net N$1: track 0.00 -> 6.87 mm
- net N$3: track 2.55 -> 8.62 mm
- net N$6: track 0.00 -> 4.93 mm
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Other:
- board text added: "RX"
- board text added: "TX"

Commit message: Terminado correciones
Parts:
- S1: device Testing:TACTILE-SWITCH-1101NE -> CaliBeta-Miselaneos:ST-SMD-6X3.5MM
- XT1: device CaliBeta-Miselaneos:CSTCE8M00G55-R0 -> CaliBeta-Miselaneos:CSTCE
Connections:
- net GND: now also S1.1; no longer S1.P$1
- net RST: now also S1.2; no longer S1.P$2
Routing:
- net VCC: track 34.8 -> 143.9 mm, vias 1 -> 6
- net GND: track 151.8 -> 253.2 mm, vias 0 -> 2
- net RST: track 28.6 -> 94.2 mm, vias 1 -> 2
- net D3: track 0.00 -> 36.7 mm, vias 0 -> 2
- net N$1: track 6.87 -> 6.37 mm
- net N$11: vias 0 -> 1
