File: Eagle/Cerradura electronica/Cerradura electronica.brd (EAGLE design)
At the start: 50 x 48.5 mm, 37 parts, among them IC1 LD117AS50TR, Q1 2N3904, Q2 IRF540N

Commit message: Add BUZZER para mejorar la funcionalidad, terminado v1.5.1
Parts:
- IC1: value LD117AS50TR -> LD1117AS50TR; device v-reg:SOT223 -> CaliBeta-IC power:SOT-223
- R7: value 150R -> 1k
- R8: value 10k -> 100k
- U$1: value A4_HORIZONTAL -> A4_H-LOGO; device Circuitos-Creativos-Estilos:LOGO -> CaliBeta-Estilos:LOGO-10MM
- XT1: device CaliBeta-Miselaneos:CSTCE -> CaliBeta-Cristales:3-SMD
- moved U$1 0.50 mm to (44.0, 11.8)
Other:
- board text added: "Desing by: CaliBeta"
- board text added: "v1.5.1"
- board text removed: "CIRCUITOS CREATIVOS"
- board text removed: "Fabricado por:"
- board text removed: "v1.5.0"
Changed lines of the file:
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@@
 </layers>
 <board>
-<fusionsync huburn="a.YnVzaW5lc3M6Z21haWwyNDYwMTM" projecturn="a.YnVzaW5lc3M6Z21haWwyNDYwMTMjMjAxOTEwMTUyMjczNDQ4MjY" f3durn="urn:adsk.wipprod:dm.lineage:JLNcbCaTSe6njw024ydtlA" pcbguid="65d882f5-96fa-496e-887d-2c29fa863bc9" lastpulledtime="" lastsyncedchangeguid="c1ef616b-cbcd-aaf2-718d-200e2dccfb05"/>
+<fusionsync huburn="a.YnVzaW5lc3M6Z21haWwyNDYwMTM" projecturn="a.YnVzaW5lc3M6Z21haWwyNDYwMTMjMjAxOTEwMTUyMjczNDQ4MjY" f3durn="urn:adsk.wipprod:dm.lineage:JLNcbCaTSe6njw024ydtlA" pcbguid="65d882f5-96fa-496e-887d-2c29fa863bc9" lastpulledtime="" lastsyncedchangeguid="e5474196-f1c3-21ba-b560-879b9e497469"/>
 <plain>
 <wire x1="48.197225" y1="49" x2="1.802775" y2="49" width="0.254" layer="20"/>
@@
 <text x="16.5" y="10.5" size="1.6764" layer="21" ratio="10" rot="R180">GND</text>
 <dimension x1="50" y1="0.5" x2="50" y2="49" x3="54.5" y3="24.75" textsize="1.778" textratio="10" layer="47"/>
-<text x="21.5" y="6" size="1.4224" layer="22" ratio="10" rot="MR180">Fabricado por:</text>
-<text x="17.5" y="3.5" size="1.4224" layer="22" ratio="10" rot="MR180">CIRCUITOS CREATIVOS</text>
-<text x="37.375" y="35.5" size="1.4224" layer="21" font="vector" ratio="10" rot="R90">1</text>
-<text x="34.75" y="35.5" size="1.4224" layer="21" font="vector" ratio="10" rot="R90">2</text>
-<text x="32.25" y="35.5" size="1.4224" layer="21" font="vector" ratio="10" rot="R90">3</text>
-<text x="29.5" y="35.5" size="1.4224" layer="21" font="vector" ratio="10" rot="R90">4</text>
-<text x="24.5" y="35.25" size="1.27" layer="21" font="vector" ratio="10">COM</text>
+<text x="27" y="4.5" size="1.778" layer="22" ratio="10" rot="MR180" align="center">Desing by:
+CaliBeta</text>
+<text x="41.375" y="35.25" size="1.4224" layer="21" font="vector" ratio="10" rot="R90">1</text>
+<text x="38.625" y="35.125" size="1.4224" layer="21" font="vector" ratio="10" rot="R90">2</text>
+<text x="36.125" y="35" size="1.4224" layer="21" font="vector" ratio="10" rot="R90">3</text>
+<text x="33.75" y="35.125" size="1.4224" layer="21" font="vector" ratio="10" rot="R90">4</text>
+<text x="30.5" y="35.5" size="1.27" layer="21" font="vector" ratio="10" align="center">COM</text>
 <text x="11" y="40.5" size="1.6764" layer="21" ratio="10" rot="R180">12V</text>
 <text x="17" y="40.5" size="1.6764" layer="21" ratio="10" rot="R180">OUT</text>
 <text x="26.5" y="8.5" size="1.778" layer="21" align="center">CERRADURA</text>
 <text x="27" y="6" size="1.778" layer="21" align="center">ELECTRONICA</text>
-<text x="27" y="3.5" size="1.778" layer="21" align="center">v1.5.0</text>
+<text x="27" y="3.5" size="1.778" layer="21" align="center">v1.5.1</text>
 <text x="44.125" y="23.75" size="1.27" layer="21" font="vector" ratio="10" rot="R270" align="center">TX</text>
 <text x="44.125" y="21.375" size="1.27" layer="21" font="vector" ratio="10" rot="R270" align="center">RX</text>
@@
 <attribute name="VALUE" x="39.54" y="12.23" size="1.27" layer="27" rot="R90"/>
 </element>
-<element name="SV1" library="con-lstb" library_urn="urn:adsk.eagle:library:162" package="MA04-1" package3d_urn="urn:adsk.eagle:package:8337/1" value="" x="46.625" y="22.5" smashed="yes" rot="R270">
+<element name="SV1" library="con-lstb" library_urn="urn:adsk.eagle:library:162" package="MA04-1" package3d_urn="urn:adsk.eagle:package:8337/1" override_package3d_urn="urn:adsk.eagle:package:14744829/2" override_package_urn="urn:adsk.eagle:footprint:8285/1" value="" x="46.625" y="22.5" smashed="yes" rot="R270">
 <attribute name="MF" value="" x="70.125" y="37.5" size="1.778" layer="27" rot="R270" display="off"/>
 <attribute name="MPN" value="" x="70.125" y="37.5" size="1.778" layer="27" rot="R270" display="off"/>
@@
 <attribute name="VALUE" x="23.96" y="28.27" size="1.27" layer="27" rot="R270"/>
 </element>
-<element name="U$1" library="Circuitos-Creativos-Estilos" package="LOGO" value="A4_HORIZONTAL" x="44" y="11.25" smashed="yes" rot="R270"/>
+<element name="U$1" library="CaliBeta-Estilos" package="LOGO-10MM" value="A4_H-LOGO" x="44" y="11.75" smashed="yes" rot="R270"/>
 <element name="Q1" library="CaliBeta-Transistores" library_urn="urn:adsk.eagle:library:14361247" package="SOT-23_BEC" package3d_urn="urn:adsk.eagle:package:14361264/3" value="2N3904" x="12.5" y="21" smashed="yes" rot="R90">
 <attribute name="NAME" x="14.655" y="21.905" size="1.27" layer="25" ratio="10" rot="R270"/>
@@
 <attribute name="VALUE" x="27.77" y="16.04" size="1.27" layer="27" rot="R180"/>
 </element>
-<element name="IC1" library="v-reg" library_urn="urn:adsk.eagle:library:409" package="SOT223" package3d_urn="urn:adsk.eagle:package:30370/1" value="LD117AS50TR" x="11.5" y="14.5" smashed="yes" rot="R270">
+<element name="IC1" library="CaliBeta-IC power" library_urn="urn:adsk.eagle:library:14742817" package="SOT-223" package3d_urn="urn:adsk.eagle:package:14742823/2" value="LD1117AS50TR" x="11.5" y="14.5" smashed="yes" rot="R270">
 <attribute name="NAME" x="13.96" y="17.0508" size="1.27" layer="25" ratio="10"/>
-<attribute name="POPULARITY" value="0" x="11.5" y="14.5" size="1.778" layer="27" rot="R270" display="off"/>
 <attribute name="VALUE" x="10.1792" y="17.04" size="1.27" layer="27" rot="R270"/>
 </element>
@@
 <attribute name="VALUE" x="6.42" y="-1.215" size="1.778" layer="27" ratio="10"/>
 </element>
-<element name="R7" library="CaliBeta-RCL" library_urn="urn:adsk.eagle:library:14345719" package="R0805" package3d_urn="urn:adsk.eagle:package:14345749/1" value="150R" x="19" y="13.5" smashed="yes" rot="R90">
+<element name="R7" library="CaliBeta-RCL" library_urn="urn:adsk.eagle:library:14345719" package="R0805" package3d_urn="urn:adsk.eagle:package:14345749/1" value="1k" x="19" y="13.5" smashed="yes" rot="R90">
 <attribute name="NAME" x="17.73" y="12.48" size="1.27" layer="25" ratio="10" rot="R90"/>
 <attribute name="VALUE" x="21.54" y="12.23" size="1.27" layer="27" rot="R90"/>
 </element>
-<element name="R8" library="CaliBeta-RCL" library_urn="urn:adsk.eagle:library:14345719" package="R0805" package3d_urn="urn:adsk.eagle:package:14345749/1" value="10k" x="19" y="20" smashed="yes" rot="R90">
+<element name="R8" library="CaliBeta-RCL" library_urn="urn:adsk.eagle:library:14345719" package="R0805" package3d_urn="urn:adsk.eagle:package:14345749/1" value="100k" x="19" y="20" smashed="yes" rot="R90">
 <attribute name="NAME" x="17.855" y="22.27" size="1.27" layer="25" ratio="10"/>
 <attribute name="VALUE" x="21.54" y="18.73" size="1.27" layer="27" rot="R90"/>
@@
 <attribute name="VALUE" x="16.58" y="50.715" size="1.778" layer="27" ratio="10" rot="R180"/>
 </element>
-<element name="TECLADO" library="con-lstb" library_urn="urn:adsk.eagle:library:162" package="MA07-1" package3d_urn="urn:adsk.eagle:package:8341/1" value="" x="33" y="38" smashed="yes">
+<element name="TECLADO" library="con-lstb" library_urn="urn:adsk.eagle:library:162" package="MA07-1" package3d_urn="urn:adsk.eagle:package:8341/1" override_package3d_urn="urn:adsk.eagle:package:14744917/2" override_package_urn="urn:adsk.eagle:footprint:8291/1" value="" x="33" y="38" smashed="yes">
 <attribute name="MF" value="" x="33" y="38" size="1.778" layer="27" display="off"/>
 <attribute name="MPN" value="" x="33" y="38" size="1.778" layer="27" display="off"/>
@@
 <attribute name="VALUE" x="34.5" y="35.4" size="1.27" layer="27" font="vector" ratio="12" rot="R180" align="bottom-center"/>
 </element>
-<element name="XT1" library="CaliBeta-Miselaneos" library_urn="urn:adsk.eagle:library:14357685" package="CSTCE" package3d_urn="urn:adsk.eagle:package:14357744/2" value="8MHz" x="42.5" y="32.5" smashed="yes" rot="R270">
+<element name="XT1" library="CaliBeta-Cristales" library_urn="urn:adsk.eagle:library:14744356" package="3-SMD" package3d_urn="urn:adsk.eagle:package:14744359/3" value="8MHz" x="42.5" y="32.5" smashed="yes" rot="R270">
 <attribute name="NAME" x="40.062" y="34.072" size="1.27" layer="25" rot="R270"/>
 <attribute name="VALUE" x="40.002" y="35.074" size="1.27" layer="27" rot="R270"/>
@@
 </drawing>
 <compatibility>
+<note version="6.3" minversion="6.2.2" severity="warning">
+Since Version 6.2.2 text objects can contain more than one line,
+which will not be processed correctly with this version.
+</note>
 <note version="8.2" severity="warning">
 Since Version 8.2, EAGLE supports online libraries. The ids
@@
 packages will not be understood (or retained) with this version.
 </note>
+<note version="9.4" severity="warning">
+Since Version 9.4, EAGLE supports the overriding of 3D packages
+in schematics and board files. Those overridden 3d packages
+will not be understood (or retained) with this version.
+</note>
 </compatibility>
